Commit message: Add files via upload

File: urdf/d435i_mount_macro.xacro (robot description, xacro)
@@ -2,8 +2,9 @@
 <robot name="mounted_camera" xmlns:xacro="http://ros.org/wiki/xacro">
 <xacro:macro name="mounted_camera" params="prefix">
-    <!-- Robot -->
+    <!-- Mount-->
     <xacro:include filename="$(find tic_tac_toe)/urdf/mount_macro.xacro" />
-    <!-- Table -->
+    <!-- Camera -->
     <xacro:include filename="$(find realsense2_description)/urdf/_d435i.urdf.xacro" />
+    <xacro:arg name="use_nominal_extrinsics" default="false"/>
     <!-- Build Kinematic Chain using imported components -->
     <xacro:camera_mount prefix=""/>

File: urdf/mount_macro.xacro (robot description, xacro)
@@ -7,5 +7,5 @@
             <origin xyz="0 0 0" rpy="0 0 0" />
             <geometry>
-                <mesh filename="package://tic_tac_toe/meshes/camera_mount_small.stl"/>
+                <mesh filename="package://tic_tac_toe/meshes/camera_mount.stl"/>
             </geometry>
             <material name="white">
@@ -16,5 +16,5 @@
             <origin xyz="0 0 0" rpy="0 0 0" />
             <geometry>
-                <mesh filename="package://tic_tac_toe/meshes/camera_mount_small.stl"/>
+                <mesh filename="package://tic_tac_toe/meshes/camera_mount.stl"/>
             </geometry>
         </collision>

Commit message: URDF Refactor
Updates should not effect external calls or usage of URDF. All outward facing named elements are named the same. Collision environment unchanged.

* Simplify to 2 macro elements and 1 xacro
* Remove support for just the MH5L less table
* Reorient mesh elements

* Update test / visualization launch files to use remaining Xacro file

File: urdf/d435i_mount_macro.xacro (robot description, xacro)
@@ -2,19 +2,34 @@
 <robot name="mounted_camera" xmlns:xacro="http://ros.org/wiki/xacro">
 <xacro:macro name="mounted_camera" params="prefix">
-    <!-- Mount-->
-    <xacro:include filename="$(find tic_tac_toe)/urdf/mount_macro.xacro" />
+    <!-- AIMS Lab Custom Camera Mount -->
+    <link name="${prefix}mount_link">
+        <visual>
+            <origin xyz="0 0 0" rpy="0 0 0" />
+            <geometry>
+                <mesh filename="package://tic_tac_toe/meshes/visual/link_4_r_camera_mount.stl"/>
+            </geometry>
+            <material name="white">
+              <color rgba="0.9 0.9 0.9 1" />
+            </material>
+        </visual>
+        <collision>
+            <origin xyz="0 0 0" rpy="0 0 0" />
+            <geometry>
+                <mesh filename="package://tic_tac_toe/meshes/collision/link_4_r_camera_mount.stl"/>
+            </geometry>
+        </collision>
+    </link>
     <!-- Camera -->
     <xacro:include filename="$(find realsense2_description)/urdf/_d435i.urdf.xacro" />
     <xacro:arg name="use_nominal_extrinsics" default="false"/>
-    <!-- Build Kinematic Chain using imported components -->
-    <xacro:camera_mount prefix=""/>
-    <link name="camera_base_link" />
-    <xacro:sensor_d435i parent="camera_base_link" use_nominal_extrinsics="$(arg use_nominal_extrinsics)">
+    <link name="tool0_camera" />
+    <xacro:sensor_d435i parent="tool0_camera" use_nominal_extrinsics="$(arg use_nominal_extrinsics)">
         <origin xyz="0 0 0" rpy="0 0 0"/>
     </xacro:sensor_d435i>
-    <joint name="mount_link-camera_base_link" type="fixed">
-        <origin xyz="0.03495 0.013 0.039" rpy="${-pi/2} 0 ${-pi/2}"/>
+    <!-- Locating: Camera mounted on lower side of Link R. Reference frame along link centerline. -->
+    <joint name="mount_link-tool0_camera" type="fixed">
+        <origin xyz="0.02195 0 -0.0535" rpy="0 ${pi/2} 0"/>
         <parent link="mount_link"/>
-        <child link="camera_base_link"/>
+        <child link="tool0_camera"/>
     </joint>
 </xacro:macro>

File: urdf/mh5l_d435i_pgn64_table_macro.xacro (robot description, xacro)
@@ -2,16 +2,15 @@
 <robot name="robot_mh5l_d435i_pgn64_table" xmlns:xacro="http://ros.org/wiki/xacro">
 <xacro:macro name="robot_mh5l_d435i_pgn64_table" params="prefix">
-    <!-- Robot w/ table and gripper -->
+    <!-- Robot w/ table and gripper --><!-- Pulled from AIMS-ROBOT-ALL Metapackage -->
     <xacro:include filename="$(find mh5l_table)/urdf/mh5l_pgn64_table_macro.xacro" />
+    <xacro:robot_mh5l_pgn64_table prefix=""/>
     <!--Camera w/ Mount -->
     <xacro:include filename="$(find tic_tac_toe)/urdf/d435i_mount_macro.xacro" />
-    <!-- Build Kinematic Chain using imported components -->
-    <xacro:robot_mh5l_pgn64_table prefix=""/>
     <xacro:mounted_camera prefix=""/>
-    <joint name="link_4_r-robot_mount" type="fixed">
-        <!--origin xyz="0.33 0 -0.09" rpy="0 ${pi/2} 0"/-->
-        <origin xyz="0.31 0 -0.051 " rpy="${pi/2} 0 0"/>
+    <!-- Join imported components -->
+    <joint name="link_4_r-mount_link" type="fixed">
+        <origin xyz="0.31 0 -0.051 " rpy="0 0 0"/>
         <parent link="link_4_r"/>
-        <child link="robot_mount"/>
+        <child link="mount_link"/>
     </joint>
 </xacro:macro>
